File: kicad/electrometer/electrometer.kicad_sch (KiCad schematic)
At the start: 0 parts

Commit message: updated pcb schematic. should fit back of disk now
Parts:
- added C2, C3: 1e-03, Capacitor_SMD:C_1206_3216Metric_Pad1.33x1.80mm_HandSolder, symbol Device:C
- added J1: Screw_Terminal_01x04, TerminalBlock_Phoenix:TerminalBlock_Phoenix_MPT-0,5-4-2.54_1x04_P2.54mm_Horizontal, symbol Connector:Screw_Terminal_01x04
- added J2: Screw_Terminal_01x02, TerminalBlock_Phoenix:TerminalBlock_Phoenix_MPT-0,5-2-2.54_1x02_P2.54mm_Horizontal, symbol Connector:Screw_Terminal_01x02
- added J3, J4: Conn_01x03_Male, Connector_PinHeader_2.54mm:PinHeader_1x03_P2.54mm_Vertical, symbol Connector:Conn_01x03_Male
- added M1: CD4051B, Package_DIP:DIP-16_W7.62mm, symbol Analog_Switch:CD4051B
- added R2, R5: 1e+03, Resistor_SMD:R_1206_3216Metric_Pad1.30x1.75mm_HandSolder, symbol Device:R_US
- added R3: 100e+03, Resistor_SMD:R_1206_3216Metric_Pad1.30x1.75mm_HandSolder, symbol Device:R_US
- added R4, R6, R7, R8: 10e+03, Resistor_SMD:R_1206_3216Metric_Pad1.30x1.75mm_HandSolder, symbol Device:R_US
- added U1: LMC6082, Package_DIP:DIP-8-16_W7.62mm, symbol Amplifier_Operational:LMC6082
Connections:
- new net: M1.1 (X4), R3.1
- new net: R2.2, R3.2, R4.2, R5.2, U1.6 (-)
- new net: C2.1, J1.1 (Pin_1), J3.1 (Pin_1), J3.2 (Pin_2), J3.3 (Pin_3), M1.16 (VDD), U1.8 (V+)
- new net: J4.2 (Pin_2), M1.10 (B), R7.1
- new net: J4.1 (Pin_1), M1.11 (A), R8.1
- new net: M1.12 (X3), M1.13 (X0), M1.14 (X1), M1.2 (X6), M1.4 (X7), M1.5 (X5), R5.1
- new net: M1.15 (X2), R4.1
- new net: J2.1 (Pin_1), M1.3 (X), U1.7
- new net: C3.2, J1.3 (Pin_3), M1.7 (VEE), U1.4 (V-)
- new net: J4.3 (Pin_3), M1.9 (C), R6.1
- new net: R2.1, U1.1
- new net GND: C2.2, C3.1, J1.2 (Pin_2), J2.2 (Pin_2), M1.6 (INH), M1.8 (VSS), R6.2, R7.2, R8.2, U1.3 (+), U1.5 (+)
- no-connect marks 0 -> 2
