File: kicad/electrometer/_autosave-electrometer.kicad_sch (KiCad schematic)
At the start: 6 parts, among them J1 Screw_Terminal_01x04, U1 LMC6082

Commit message: updated board
Parts:
- U1: footprint Package_DIP:DIP-8-16_W7.62mm -> Package_DIP:DIP-8_W7.62mm
Changed lines of the file:
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@@
 			)
 		)
-		(property "Footprint" "Package_DIP:DIP-8-16_W7.62mm"
+		(property "Footprint" "Package_DIP:DIP-8_W7.62mm"
 			(at 41.91 144.78 0)
 			(effects
@@
 			)
 		)
-		(property "Footprint" "Package_DIP:DIP-8-16_W7.62mm"
+		(property "Footprint" "Package_DIP:DIP-8_W7.62mm"
 			(at 78.74 144.78 0)
 			(effects
