File: kicad/ADC/ADC_and_voltage_boost/ADC_and_voltage_boost.kicad_pcb (KiCad board)
At the start: 2 copper layers, 29.7 x 43.4 mm, 10 parts, among them J1 Screw_Terminal_01x04, J4 Screw_Terminal_01x02, U3 MOUDLE-SEEEDUINO-XIAO-ESP32C3, U4 MAX1032BEUG_

Commit message: updated pcb
Parts:
- removed J4: Screw_Terminal_01x02, TerminalBlock_Phoenix:TerminalBlock_Phoenix_MPT-0,5-2-2.54_1x02_P2.54mm_Horizontal
- removed the REF** at (138.9, 86.4)
- removed the REF** at (160.5, 86.4)
- added C1: 0.1e-6, Capacitor_SMD:C_0805_2012Metric, F.Cu at (144.0, 93.0)
- added C11: 0.1e-6, Capacitor_SMD:C_0805_2012Metric, F.Cu at (144.0, 95.0)
- added J2: Screw_Terminal_01x04, TerminalBlock_Phoenix:TerminalBlock_Phoenix_MPT-0,5-4-2.54_1x04_P2.54mm_Horizontal, F.Cu at (155.4, 88.9)
- added REF**: MountingHole_2.7mm_M2.5, MountingHole:MountingHole_2.7mm_M2.5, F.Cu at (139.4, 86.9)
- added REF**: MountingHole_2.7mm_M2.5, MountingHole:MountingHole_2.7mm_M2.5, F.Cu at (160.8, 86.9)
- C2, C3, C8, C9: footprint Capacitor_SMD:C_1206_3216Metric_Pad1.33x1.80mm_HandSolder -> Capacitor_SMD:C_0805_2012Metric
- moved C2 18.7 mm to (155.6, 98.6), turned to 0 degrees
- moved C8 4.03 mm to (155.7, 94.5), turned to 180 degrees
- moved J1 3.30 mm to (138.7, 92.2)
- moved C9 1.25 mm to (155.7, 96.5), turned to 180 degrees
Routing:
- net +5V: track 52.6 -> 32.9 mm, vias 0 -> 4
- net +3.3V: track 97.9 -> 88.2 mm
- net GND: track 82.0 -> 72.5 mm, vias 2 -> 3
- net Net-(U4-REF): track 7.67 -> 2.74 mm
- net Net-(J2-Pin_1): track 8.30 -> 11.3 mm
- net Net-(U4-REFCAP): track 4.60 -> 2.29 mm
- net Net-(J2-Pin_3): track 6.60 -> 7.55 mm
Other:
- board text added: "Screw_Terminal_01x04"
