File: kicad/ADC/ADC_and_voltage_boost/_autosave-ADC_and_voltage_boost.kicad_sch (KiCad schematic)
At the start: 11 parts, among them J1 Screw_Terminal_01x04, J2 Screw_Terminal_01x04, J3 Screw_Terminal_01x02, U4 MAX1032BEUG_

Commit message: fixing board issues - kicad
Connections:
- no-connect marks 5 -> 23
Changed lines of the file:
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@@
+	)
+	(no_connect
+		(at 185.42 38.1)
+	)
+	(no_connect
+		(at 185.42 15.24)
+	)
+	(no_connect
+		(at 185.42 43.18)
 	)
 	(no_connect
@@
 	)
 	(no_connect
+		(at 185.42 35.56)
+	)
+	(no_connect
+		(at 160.02 27.94)
+	)
+	(no_connect
+		(at 160.02 25.4)
+	)
+	(no_connect
+		(at 160.02 48.26)
+	)
+	(no_connect
+		(at 177.8 5.08)
+	)
+	(no_connect
+		(at 185.42 40.64)
+	)
+	(no_connect
+		(at 160.02 20.32)
+	)
+	(no_connect
+		(at 160.02 22.86)
+	)
+	(no_connect
 		(at 190.5 111.76)
+	)
+	(no_connect
+		(at 160.02 33.02)
 	)
 	(no_connect
@@
 	)
 	(no_connect
+		(at 160.02 58.42)
+	)
+	(no_connect
 		(at 190.5 114.3)
 	)
 	(no_connect
+		(at 160.02 55.88)
+	)
+	(no_connect
+		(at 185.42 22.86)
+	)
+	(no_connect
+		(at 160.02 50.8)
+	)
+	(no_connect
+		(at 160.02 30.48)
+	)
+	(no_connect
+		(at 160.02 17.78)
+	)
+	(no_connect
